File: hardware/io-4.kicad_pcb (KiCad board)
At the start: 2 copper layers, 35 x 35 mm, 28 parts, among them J1 AKL_5_2, J2 AKL_5_2, J3 AKL_5_2, J4 AKL_5_2, J5 AKL_5_2, P1 CON-SENSOR2, P2 DEBUG, P3 BOOT, U1 XMC1XXX24, U2 DRILL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

Commit message: fix status text
Other:
- board text added: "Status"
- board text removed: "status"
Changed lines of the file:
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@@
-(kicad_pcb (version 4) (host pcbnew 4.0.2+dfsg1-stable)
+(kicad_pcb (version 4) (host pcbnew 4.0.7-e2-6376~58~ubuntu17.04.1)
   (general
     (links 47)
     (no_connects 0)
-    (area 122.844999 66.044999 282.3718 165.09238)
+    (area 14.15415 66.044999 159.555001 196.440793)
     (thickness 1.6002)
     (drawings 24)
@@
       (xy 1.301301 2.715081) (xy 1.302426 2.714986)) (layer B.SilkS) (width 0.01))
   )
-  (gr_text status (at 157.49 75.1 90) (layer F.SilkS)
+  (gr_text Status (at 157.49 75.1 90) (layer F.SilkS)
     (effects (font (size 0.8 0.8) (thickness 0.15)))
   )
