File: hardware/io-4.kicad_pcb (KiCad board)
At the start: 2 copper layers, 35 x 35 mm, 28 parts, among them J1 AKL_5_2, J2 AKL_5_2, J3 AKL_5_2, J4 AKL_5_2, J5 AKL_5_2, P1 CON-SENSOR2, P2 DEBUG, P3 BOOT, U1 XMC1XXX24, U2 DRILL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

Commit message: change description text
Other:
- board text added: "Output Only"
- board text removed: "Output only"
Changed lines of the file:
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@@
     (effects (font (size 1.00076 1.00076) (thickness 0.14986)))
   )
-  (gr_text "Output only" (at 135.12302 84.3026 270) (layer F.SilkS)
+  (gr_text "Output Only" (at 135.12302 84.3026 270) (layer F.SilkS)
     (effects (font (size 0.8001 0.8001) (thickness 0.14986)))
   )

Commit message: specify processor
Parts:
- U1: value XMC1XXX24 -> XMC1100
Changed lines of the file:
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@@
       (effects (font (size 0.3 0.3) (thickness 0.075)))
     )
-    (fp_text value XMC1XXX24 (at 0 0.8 270) (layer F.Fab)
+    (fp_text value XMC1100 (at 0 0.8 270) (layer F.Fab)
       (effects (font (size 0.3 0.3) (thickness 0.075)))
     )

Commit message: specify led color
Parts:
- D1: value LED -> blue
Changed lines of the file:
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@@
       (effects (font (size 0.2 0.2) (thickness 0.05)))
     )
-    (fp_text value LED (at 0.75 0.45 90) (layer F.Fab)
+    (fp_text value blue (at 0.75 0.45 90) (layer F.Fab)
       (effects (font (size 0.2 0.2) (thickness 0.05)))
     )

Commit message: specify resistor
Parts:
- R1: value R -> 1k
Changed lines of the file:
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@@
       (effects (font (size 0.2 0.2) (thickness 0.05)))
     )
-    (fp_text value R (at 0.05 -0.375 90) (layer F.Fab)
+    (fp_text value 1k (at 0.05 -0.375 90) (layer F.Fab)
       (effects (font (size 0.2 0.2) (thickness 0.05)))
     )
