File: hardware/io4-v2.kicad_pcb (KiCad board)
At the start: 2 copper layers, 35 x 35 mm, 28 parts, among them J1 AKL_5_2, J2 AKL_5_2, J3 AKL_5_2, J4 AKL_5_2, J5 AKL_5_2, P1 CON-SENSOR2, P2 DEBUG, P3 BOOT, U1 XMC1100, U2 DRILL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

Commit message: Data Cleanup
Parts:
- moved U3 30.0 mm to (156.2, 69.4), turned to 180 degrees
- moved U5 30.0 mm to (126.2, 99.4), turned to 180 degrees
- moved U2 30.0 mm to (126.2, 69.4), turned to 90 degrees
- moved U4 30.0 mm to (156.2, 99.4), turned to 90 degrees
- moved D1 24.8 mm to (131.9, 69.5), turned to 180 degrees
- moved P1 24.7 mm to (141.2, 66.9), turned to 180 degrees
- moved Fiducial_Mark 23.2 mm to (151.2, 71.4), turned to 90 degrees
- moved R1 23.2 mm to (131.9, 70.9), turned to 180 degrees
- moved Ref** 23.0 mm to (148.4, 95.6)
- moved Fiducial_Mark 23.0 mm to (130.2, 96.4), turned to 90 degrees
- moved J2 18.0 mm to (152.9, 89.4), turned to -90 degrees
- moved J3 18.0 mm to (129.5, 89.4), turned to 90 degrees
- moved J1 18.0 mm to (152.9, 79.4), turned to -90 degrees
- moved J4 18.0 mm to (129.5, 79.4), turned to 90 degrees
- moved C1 16.7 mm to (137.0, 73.4), turned to 180 degrees
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Routing:
- net GND: track 26.0 -> 24.4 mm
- net Net-(P3-Pad2): track 2.16 -> 1.35 mm
Other:
- net class Default removed
- board text added: "Copyright Tinkerforge GmbH 2023. This documentation describes Open Hardware and is licensed under the CERN OHL v. 1.1. You may redistribute and modify this documentation under the terms of the CERN OHL v.1.1. (http://ohwr.org/cernohl). This documentation is distributed WITHOUT ANY EXPRESS OR IMPLIED WARRANTY, INCLUDING OF MERCHANTABILITY, SATISFACTORY QUALITY AND FITNESS FOR A PARTICULAR PURPOSE.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"
- board text added: "IO-4 2.0"
- board text removed: "2.0"
- board text removed: "Copyright Tinkerforge GmbH 2018. This documentation describes Open Hardware and is licensed under the CERN OHL v. 1.1. You may redistribute and modify this documentation under the terms of the CERN OHL v.1.1. (http://ohwr.org/cernohl). This documentation is distributed WITHOUT ANY EXPRESS OR IMPLIED WARRANTY, INCLUDING OF MERCHANTABILITY, SATISFACTORY QUALITY AND FITNESS FOR A PARTICULAR PURPOSE.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"
- board text removed: "IO-4"
